File: Eagle/various/various.brd (EAGLE design)
At the start: 99.8 x 82 mm, 24 parts, among them Q1 2N5088

Commit message: Eagle
Parts:
- removed C1, C2: 10uF, SparkFun-Capacitors:CPOL-RADIAL-2.5MM-5MM
- removed Q1: 2N5088, transistor-npn:TO92
- removed R3: 1K, resistor:0207/12
- removed R5: 10K, resistor:0207/12
- added J11, J8: (no value), SparkFun-Connectors:1X01
- added J18, J19: (no value), SparkFun-Connectors:1X05
- added J27: (no value), SparkFun-Connectors:1X11
- added J31: (no value), SparkFun-Connectors:1X14
- added J32: (no value), SparkFun-Connectors:1X10
- added JP19, JP3, JP4, JP5, JP7: (no value), SparkFun-Connectors:1X15
- added S1: (no value), switch-omron:B3F-40XX
- J1, J2: device SparkFun-Connectors:1X20 -> SparkFun-Connectors:1X04
- moved J41 77.7 mm to (20.3, 76.7)
- moved J2 69.1 mm to (6.35, 6.35), turned to 90 degrees
- moved J3 67.5 mm to (44.7, 14.7)
- moved J6 63.5 mm to (2.03, 14.1)
- moved J7 63.5 mm to (2.03, 8.89)
- moved J40 60.0 mm to (27.4, 67.8), turned to 180 degrees
- moved J39 58.9 mm to (20.3, 69.1)
- moved J5 53.7 mm to (53.6, 8.38)
- moved J4 53.2 mm to (53.6, 13.6)
- moved J42 41.5 mm to (93.5, 22.6), turned to 180 degrees
- moved J43 34.9 mm to (37.6, 65.5)
- moved J34 33.1 mm to (37.6, 58.4)
- moved J37 30.4 mm to (30.0, 68.1), turned to 0 degrees
- moved JP14 26.7 mm to (36.3, 55.6)
- moved S2 22.4 mm to (90.9, 76.7)
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Connections:
- removed net 3.3V: J2.1
- removed net 3.3V2: C2.1
- removed net 3.3V_E: C1.1, Q1.1
- removed net GND2: C2.2
- removed net GND_E: C1.2, R5.1
- removed net GPIO05: J2.15
- removed net GPIO06: J2.16, J3.1
- removed net GPIO12: J1.5
- removed net GPIO13: J2.17, J3.2
- removed net GPIO16: J1.3
- removed net GPIO19: J2.18, J3.3
- removed net GPIO20: J1.2
- removed net GPIO21: J1.1
- removed net GPIO26: J2.19, J3.4
- removed net N$1: J1.16
- removed net N$4: Q1.2, R3.2
- removed net RX5_E: R3.1
- removed net RX_E: Q1.3
- removed net TXD0: J1.17
- new net A1_D: J18.4, JP3.5
- new net A2_D: J18.3, JP3.6
- new net A3_D: J19.4, JP3.7
- new net A4_D: J19.3, JP3.8
- new net A6_D: JP3.10
- new net D0: J3.2, JP5.2
- new net D1: JP5.1
- new net D10: J2.1, JP5.13
- new net D10_D: JP4.13
- new net D11: J27.10, JP5.14
- new net D11_D: JP4.14
- new net D12: J27.11, JP5.15
- new net D12_D: JP4.15
- new net D13: JP7.1
- new net D13_D: JP3.1
- new net D14: JP7.4
- new net D15: JP7.5
- new net D16: JP7.6
- new net D17: J27.5, JP7.7
- new net D18: JP7.8
- new net D19: JP7.9
- new net D2: J27.6, JP5.5
- new net D20: JP7.10
- new net D21: JP7.11
- new net D2_D: JP4.5, S1.3
- new net D3: J27.4, JP5.6
- new net D4: J27.7, JP5.7
- new net D5: J2.4, JP5.8
- new net D6: J2.3, JP5.9
- new net D6_D: J18.5, J19.5, JP4.9
- new net D7: J27.9, JP5.10
- new net D8: J27.8, JP5.11
- new net D9: J2.2, JP5.12
- new net D9_D: JP4.12
- new net RX_D: JP4.2
- new net TX_D: J1.4, JP4.1
- new net VCC_D: J1.1, J11.1, J18.2, J19.2, JP3.12
- net 7.4V: now also J27.3
- net D3_D: now also JP4.6
- net GND: now also J27.1, J3.3, JP5.4, JP7.14; no longer J1.18, J2.5
- net GND_D: now also J1.2, J18.1, J19.1, J8.1, JP3.14, JP4.4, S1.1
- net VCC: now also J27.2, J3.4, JP7.12; no longer J1.20
Other:
- board size 99.8 x 82 mm -> 99.8 x 85.1 mm
- board text added: "HC-06"
- board text removed: "+"
- board text removed: "10 K"
- board text removed: "1K"
- board text removed: "Prog"
- board text removed: "RTxGn5V"
- board text removed: "VCC"
- board text removed: "Wemos"
