File: Eagle/piHatJoystick/piHatJoystick.brd (EAGLE design)
At the start: 99.1 x 85.6 mm, 49 parts, among them J17 Relay, J20 Pixel, J22 IR Rx, X1 53047-11

Commit message: Binary numbers
Parts:
- added J29: (no value), SparkFun-Connectors:1X06_NO_SILK
- added J30: (no value), SparkFun-Connectors:1X01
- added Q1, Q2: 2N5088, transistor-npn:TO92
- added R1, R3: 1K, resistor-power:CA0001
- added R2: 10K, resistor-power:CA0001
- added R4: 200ohm, resistor-power:CA0001
- moved J41 77.7 mm to (60.5, 10.4)
- moved J34 76.0 mm to (61.0, 2.03), turned to 90 degrees
- moved J24 75.4 mm to (19.6, 63.8)
- moved J42 46.3 mm to (51.1, 18.0)
- moved J38 44.2 mm to (93.0, 4.06)
- moved J16 11.5 mm to (21.6, 27.2)
- moved J31 7.62 mm to (97.3, 10.2)
- moved J43 6.59 mm to (14.5, 77.5)
- moved J5 5.92 mm to (56.6, 3.30)
- moved J4 5.64 mm to (56.6, 8.89)
- moved X1 5.61 mm to (15.5, 34.8)
- moved J3 4.89 mm to (49.0, 12.4)
- moved J40 4.23 mm to (53.3, 18.0)
- moved J20 2.97 mm to (3.05, 44.2)
- moved J17 1.27 mm to (28.4, 39.6)
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Connections:
- new net A1_B: J14.5, R1.1
- new net D2_B: J15.5, J25.6
- new net D4_B: J15.7, J25.5
- new net GPIO12: J9.5, Q1.3, R2.2
- new net GPIO13: J10.18
- new net GPIO16: J14.4, J9.3
- new net GPIO19: J10.19
- new net GPIO20: J25.3, J29.5, J9.2
- new net GPIO21: J25.2, J29.2, J9.1
- new net GPIO26: J10.20
- new net GPIO5: J10.16, J25.1, J29.1
- new net GPIO6: J10.17
- new net N$1: Q1.2, R1.2
- new net N$2: Q2.2, R3.2
- new net N$4: Q2.3, R4.1
- new net TX_C: J21.1, R4.2
- net 3.3V_B: now also Q1.1
- net 5V_C: now also Q2.1
- net GND_B: now also J25.4, J29.4, J29.6, R2.1
- net TXIR_C: now also R3.1; no longer J21.1
- net VCC_B: now also J29.3
Routing:
- net GPIO21: track 0.00 -> 128.8 mm, vias 0 -> 1
- net GND_B: track 0.00 -> 124.0 mm
- net GPIO12: track 0.00 -> 108.0 mm, vias 0 -> 1
- net GND_D: track 0.00 -> 106.5 mm
- net VCC_B: track 0.00 -> 102.9 mm
- net GND: track 0.00 -> 79.4 mm
- net GPIO5: track 0.00 -> 74.5 mm
- net VCC_D: track 0.00 -> 74.3 mm
- net GND_C: track 0.00 -> 72.3 mm
- net GPIO20: track 0.00 -> 68.9 mm, vias 0 -> 2
- net D6_D: track 0.00 -> 68.4 mm
- net VCC: track 0.00 -> 57.1 mm
- net 7V_B: track 0.00 -> 55.1 mm
- net 3.3V_B: track 0.00 -> 52.6 mm, vias 0 -> 1
- net 5V_C: track 0.00 -> 51.8 mm
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Other:
- board text added: "10K"
- board text added: "1K"
- board text added: "200"
