File: Eagle/piHatJoystick/piHatJoystick.sch (EAGLE design)
At the start: 38 parts, among them J17 Relay, J20 Pixel, J22 IR Rx, X1 53047-11

Commit message: Binary numbers
Parts:
- added J29: (no value), SparkFun-Connectors:CONN_06NO_SILK_FEMALE_PTH
- added J30: (no value), SparkFun-Connectors:CONN_01
- added Q1, Q2: 2N5088, transistor-npn:2N5088
- added R1, R3: 1K, resistor-power:RCA0001
- added R2: 10K, resistor-power:RCA0001
- added R4: 200ohm, resistor-power:RCA0001
Connections:
- new net A1_B: J14.5, R1.1
- new net D2_B: J15.5, J25.6
- new net D4_B: J15.7, J25.5
- new net GPIO12: J9.5, Q1.E, R2.2
- new net GPIO13: J10.18
- new net GPIO16: J14.4, J9.3
- new net GPIO19: J10.19
- new net GPIO20: J25.3, J29.5, J9.2
- new net GPIO21: J25.2, J29.2, J9.1
- new net GPIO26: J10.20
- new net GPIO5: J10.16, J25.1, J29.1
- new net GPIO6: J10.17
- new net N$1: Q1.B, R1.2
- new net N$2: Q2.B, R3.2
- new net N$4: Q2.E, R4.1
- new net TX_C: J21.1, R4.2
- net 3.3V_B: now also Q1.C
- net 5V_C: now also Q2.C
- net GND_B: now also J25.4, J29.4, J29.6, R2.1
- net TXIR_C: now also R3.1; no longer J21.1
- net VCC_B: now also J29.3
Other:
- note added: "Fire"
- note added: "Hit Detected"
- note added: "Pixels (D2)"
- moved on the sheet: J12, J13
