File: Eagle/nanoHC06Rx/nanoHC06Rx.sch (EAGLE design)
At the start: 55 parts, among them J10 Relay, J14 Relay, J16 Relay, J17 Relay, J2 Relay, J33 Relay, J41 Relay, J43 Relay, Q1 2N5088

Commit message: yo
Parts:
- added J44, J45, J46, J47: (no value), SparkFun-Connectors:CONN_01PTH_2MM
Connections:
- net BATT3.3V_B: now also J46.1
- net BATT_3V3_D: now also J44.1
- net GND_B: now also J47.1
- net GND_D: now also J45.1
Changed lines of the file:
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@@
 <part name="J41" library="SparkFun-Connectors" deviceset="CONN_03" device="" value="Relay"/>
 <part name="J43" library="SparkFun-Connectors" deviceset="CONN_03" device="" value="Relay"/>
+<part name="J44" library="SparkFun-Connectors" library_urn="urn:adsk.eagle:library:513" deviceset="CONN_01" device="PTH_2MM" package3d_urn="urn:adsk.eagle:package:38029/1"/>
+<part name="J45" library="SparkFun-Connectors" library_urn="urn:adsk.eagle:library:513" deviceset="CONN_01" device="PTH_2MM" package3d_urn="urn:adsk.eagle:package:38029/1"/>
+<part name="J46" library="SparkFun-Connectors" library_urn="urn:adsk.eagle:library:513" deviceset="CONN_01" device="PTH_2MM" package3d_urn="urn:adsk.eagle:package:38029/1"/>
+<part name="J47" library="SparkFun-Connectors" library_urn="urn:adsk.eagle:library:513" deviceset="CONN_01" device="PTH_2MM" package3d_urn="urn:adsk.eagle:package:38029/1"/>
 </parts>
 <sheets>
@@
 <attribute name="NAME" x="-1.27" y="250.952" size="1.778" layer="95" font="vector" rot="R180"/>
 </instance>
+<instance part="J44" gate="G$1" x="214.63" y="355.6" smashed="yes" rot="R180">
+<attribute name="VALUE" x="217.17" y="360.426" size="1.778" layer="96" font="vector" rot="R180"/>
+<attribute name="NAME" x="217.17" y="352.552" size="1.778" layer="95" font="vector" rot="R180"/>
+</instance>
+<instance part="J45" gate="G$1" x="326.39" y="361.95" smashed="yes">
+<attribute name="VALUE" x="323.85" y="357.124" size="1.778" layer="96" font="vector"/>
+<attribute name="NAME" x="323.85" y="364.998" size="1.778" layer="95" font="vector"/>
+</instance>
+<instance part="J46" gate="G$1" x="-31.75" y="255.27" smashed="yes" rot="R180">
+<attribute name="VALUE" x="-29.21" y="260.096" size="1.778" layer="96" font="vector" rot="R180"/>
+<attribute name="NAME" x="-29.21" y="252.222" size="1.778" layer="95" font="vector" rot="R180"/>
+</instance>
+<instance part="J47" gate="G$1" x="200.66" y="265.43" smashed="yes">
+<attribute name="VALUE" x="198.12" y="260.604" size="1.778" layer="96" font="vector"/>
+<attribute name="NAME" x="198.12" y="268.478" size="1.778" layer="95" font="vector"/>
+</instance>
 </instances>
 <busses>
@@
 <label x="196.85" y="401.32" size="1.778" layer="95" rot="R90"/>
 </segment>
+<segment>
+<pinref part="J45" gate="G$1" pin="1"/>
+<wire x1="334.01" y1="361.95" x2="337.82" y2="361.95" width="0.1524" layer="91"/>
+<label x="336.55" y="361.95" size="1.778" layer="95"/>
+</segment>
 </net>
 <net name="VCC_D" class="0">
@@
 <label x="-20.32" y="254" size="1.778" layer="95"/>
 </segment>
+<segment>
+<pinref part="J47" gate="G$1" pin="1"/>
+<wire x1="208.28" y1="265.43" x2="215.9" y2="265.43" width="0.1524" layer="91"/>
+<label x="215.9" y="265.43" size="1.778" layer="95"/>
+</segment>
 </net>
 <net name="VCC_B" class="0">
@@
 <label x="-45.72" y="285.75" size="1.778" layer="95"/>
 </segment>
+<segment>
+<pinref part="J46" gate="G$1" pin="1"/>
+<wire x1="-39.37" y1="255.27" x2="-53.34" y2="255.27" width="0.1524" layer="91"/>
+<label x="-53.34" y="255.27" size="1.778" layer="95"/>
+</segment>
 </net>
 <net name="BATT_3V3_D" class="0">
@@
 <label x="231.14" y="402.59" size="1.778" layer="95"/>
 </segment>
-</net>
+<segment>
+<pinref part="J44" gate="G$1" pin="1"/>
+<wire x1="207.01" y1="355.6" x2="191.77" y2="355.6" width="0.1524" layer="91"/>
+<label x="191.77" y="355.6" size="1.778" layer="95"/>
+</segment>
+</net>

Commit message: Requirements
Parts:
- removed C1: 10uF, SparkFun-Capacitors:10UF-POLAR-RADIAL-2.5MM-KIT-25V-20%
- removed J20: (no value), SparkFun-Connectors:CONN_06NO_SILK_FEMALE_PTH
- removed J22, J24, J28, J36: (no value), SparkFun-Connectors:CONN_01
- removed J27: (no value), SparkFun-Connectors:CONN_11
- removed J46, J47: (no value), SparkFun-Connectors:CONN_01PTH_2MM
- removed PROG1: (no value), SparkFun-Connectors:CONN_02
- removed U$1: V_REG_LD1117VXX, SparkFun-IC-Power:V_REG_LD1117VXX
- added D1, D2, D3, D4, D5, D6: 1N5333, diode:1N5333
- added J48: (no value), SparkFun-Connectors:CONN_04
- J21: device SparkFun-Connectors:CONN_01 -> SparkFun-Connectors:CONN_04
Connections:
- removed net BATT3.3V_B: J22.1, J24.1, J46.1
- new net N$2: D1.A, J16.2
- new net N$4: D2.A, J17.2
- new net N$5: D3.A, J41.2
- new net N$6: D4.A, J43.2
- new net N$7: D5.A, J2.2
- new net N$8: D6.A, J33.2
- net 3.3V_B: no longer C1.+, J36.1, PROG1.1, PROG1.2, U$1.OUT
- net 5V_B: now also D1.C, D2.C, D3.C, D4.C, J21.1; no longer J16.2, J17.2, J20.3, J41.2, J43.2, U$1.IN
- net 7.4V: no longer J27.3
- net D10_D: now also J48.1
- net D11: no longer J27.10
- net D11_D: now also J48.3
- net D12: no longer J27.11
- net D12_D: now also J48.4
- net D17: no longer J27.5
- net D2: no longer J27.6
- net D3: no longer J27.4
- net D4: no longer J27.7
- net D7: no longer J27.9
- net D8: no longer J27.8
- net GND: no longer J27.1
- net GND_B: now also J15.2, J21.2; no longer C1.-, J20.4, J20.6, J21.1, J47.1, U$1.GND
- net GPIO02_B: now also J16.3; no longer J20.5
- net GPIO04_B: now also J21.4
- net GPIO14_B: now also J43.1; no longer J20.1
- net GPIO15_B: no longer J12.3, J20.2, J43.1
- net GPIO16_B: no longer J16.3, J28.1
- net UOT: now also J21.3
- net VCC: now also D5.C, D6.C; no longer J2.2, J27.2, J33.2
- net VCC_D: now also J48.2
Other:
- note removed: "Fire Relay"
- note removed: "IR Receive"
- note removed: "IR Transmit"
- note removed: "Pixel Data"
- note removed: "Turret Down"
- note removed: "Turret Up"
- moved on the sheet: J16, J17, J2, J33, J34, J41

Commit message: arduino
Parts:
- added J20: Relay, SparkFun-Connectors:CONN_03
Connections:
- net D2: now also J20.1
- net D4: now also J3.1
- net GND: now also J20.3
- net VCC: now also J20.2
Changed lines of the file:
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@@
 <part name="D6" library="diode" library_urn="urn:adsk.eagle:library:210" deviceset="1N5333" device="" package3d_urn="urn:adsk.eagle:package:43351/1"/>
 <part name="J21" library="SparkFun-Connectors" library_urn="urn:adsk.eagle:library:513" deviceset="CONN_04" device="" package3d_urn="urn:adsk.eagle:package:38085/1"/>
+<part name="J20" library="SparkFun-Connectors" deviceset="CONN_03" device="" value="Relay"/>
+<part name="GND8" library="SparkFun" deviceset="GND" device=""/>
+<part name="P+4" library="SparkFun" deviceset="VCC" device=""/>
 </parts>
 <sheets>
@@
 </instance>
 <instance part="D5" gate="1" x="21.59" y="157.48" smashed="yes">
-<attribute name="NAME" x="19.812" y="159.385" size="1.778" layer="95"/>
+<attribute name="NAME" x="19.812" y="156.845" size="1.778" layer="95"/>
 <attribute name="VALUE" x="19.812" y="154.051" size="1.778" layer="96"/>
 </instance>
@@
 <attribute name="VALUE" x="54.61" y="291.084" size="1.778" layer="96" font="vector"/>
 <attribute name="NAME" x="54.61" y="306.578" size="1.778" layer="95" font="vector"/>
+</instance>
+<instance part="J20" gate="J$1" x="85.09" y="153.67" smashed="yes" rot="R90">
+<attribute name="VALUE" x="92.456" y="151.13" size="1.778" layer="96" font="vector" rot="R90"/>
+<attribute name="NAME" x="79.502" y="151.13" size="1.778" layer="95" font="vector" rot="R90"/>
+</instance>
+<instance part="GND8" gate="1" x="80.01" y="165.1" smashed="yes" rot="R270">
+<attribute name="VALUE" x="77.47" y="167.64" size="1.778" layer="96" rot="R270"/>
+</instance>
+<instance part="P+4" gate="1" x="85.09" y="168.91" smashed="yes">
+<attribute name="VALUE" x="84.074" y="172.466" size="1.778" layer="96"/>
 </instance>
 </instances>
@@
 <wire x1="160.02" y1="196.85" x2="163.83" y2="196.85" width="0.1524" layer="91"/>
 </segment>
+<segment>
+<pinref part="J20" gate="J$1" pin="3"/>
+<pinref part="GND8" gate="1" pin="GND"/>
+<wire x1="82.55" y1="165.1" x2="82.55" y2="161.29" width="0.1524" layer="91"/>
+</segment>
 </net>
 <net name="D3" class="0">
@@
 <wire x1="41.91" y1="157.48" x2="44.45" y2="157.48" width="0.1524" layer="91"/>
 </segment>
+<segment>
+<pinref part="J20" gate="J$1" pin="2"/>
+<pinref part="P+4" gate="1" pin="VCC"/>
+<wire x1="85.09" y1="168.91" x2="85.09" y2="161.29" width="0.1524" layer="91"/>
+</segment>
 </net>
 <net name="D4" class="0">
@@
 <label x="158.75" y="156.21" size="1.778" layer="95"/>
 </segment>
+<segment>
+<pinref part="J3" gate="G$1" pin="1"/>
+<wire x1="82.55" y1="181.61" x2="86.36" y2="181.61" width="0.1524" layer="91"/>
+<label x="86.36" y="181.61" size="1.778" layer="95"/>
+</segment>
 </net>
 <net name="D1" class="0">
@@
 <pinref part="J3" gate="G$1" pin="2"/>
 <wire x1="82.55" y1="184.15" x2="88.9" y2="184.15" width="0.1524" layer="91"/>
-<label x="92.71" y="184.15" size="1.778" layer="95"/>
+<label x="86.36" y="184.15" size="1.778" layer="95"/>
 </segment>
 </net>
@@
 <label x="5.08" y="147.32" size="1.778" layer="95"/>
 </segment>
-</net>
+<segment>
+<pinref part="J20" gate="J$1" pin="1"/>
+<wire x1="87.63" y1="161.29" x2="91.44" y2="161.29" width="0.1524" layer="91"/>
+<label x="91.44" y="161.29" size="1.778" layer="95"/>
+</segment>
+</net>
