File: Eagle/JDY-40 Joystick/nanoHC06Rx.sch (EAGLE design)
At the start: 22 parts

Commit message: Added Chrome App
Parts:
- removed U$2: 1X8, headers(2mm):1X8
- added J2: (no value), SparkFun-Connectors:CONN_03
- J1: device SparkFun-Connectors:CONN_08" -> SparkFun-Connectors:CONN_06SILK_FEMALE_PTH
Connections:
- removed net N$10: J1.6, U$2.6
- removed net N$11: J1.7, U$2.7
- removed net N$12: J1.8, U$2.8
- removed net N$5: J1.1, U$2.1
- removed net N$6: J1.2, U$2.2
- removed net N$7: J1.3, U$2.3
- removed net N$8: J1.4, U$2.4
- removed net N$9: J1.5, U$2.5
- net D7_D: now also J2.2
- net GND_D: now also J1.6, J2.1
- net RX_D: now also J1.3, JP4.1; no longer JP4.2
- net TX_D: now also J1.2, JP4.2; no longer JP4.1
- net VCC_D: now also J2.3
Changed lines of the file:
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@@
 <part name="R2" library="resistor" library_urn="urn:adsk.eagle:library:348" deviceset="R-US_" device="0309/10" package3d_urn="urn:adsk.eagle:package:26087/1"/>
 <part name="R3" library="resistor" library_urn="urn:adsk.eagle:library:348" deviceset="R-US_" device="0309/10" package3d_urn="urn:adsk.eagle:package:26087/1"/>
-<part name="U$2" library="headers(2mm)" deviceset="1X8" device=""/>
-<part name="J1" library="SparkFun-Connectors" library_urn="urn:adsk.eagle:library:513" deviceset="CONN_08" device="&quot;" package3d_urn="urn:adsk.eagle:package:38138/1"/>
+<part name="J1" library="SparkFun-Connectors" library_urn="urn:adsk.eagle:library:513" deviceset="CONN_06" device="SILK_FEMALE_PTH" package3d_urn="urn:adsk.eagle:package:38009/1"/>
+<part name="J2" library="SparkFun-Connectors" library_urn="urn:adsk.eagle:library:513" deviceset="CONN_03" device="" package3d_urn="urn:adsk.eagle:package:38063/1"/>
 </parts>
 <sheets>
@@
 <attribute name="VALUE" x="327.152" y="419.1" size="1.778" layer="96" rot="R90"/>
 </instance>
-<instance part="U$2" gate="G$1" x="247.65" y="443.23" smashed="yes" rot="R180">
-<attribute name="NAME" x="250.19" y="429.895" size="1.27" layer="95" font="vector" rot="R180"/>
-<attribute name="VALUE" x="250.19" y="455.295" size="1.27" layer="96" font="vector" rot="R180"/>
-</instance>
-<instance part="J1" gate="G$1" x="234.95" y="440.69" smashed="yes">
-<attribute name="VALUE" x="229.87" y="428.244" size="1.778" layer="96" font="vector"/>
-<attribute name="NAME" x="229.87" y="453.898" size="1.778" layer="95" font="vector"/>
+<instance part="J1" gate="G$1" x="195.58" y="426.72" smashed="yes" rot="R180">
+<attribute name="VALUE" x="200.66" y="436.626" size="1.778" layer="96" font="vector" rot="R180"/>
+<attribute name="NAME" x="200.66" y="416.052" size="1.778" layer="95" font="vector" rot="R180"/>
+</instance>
+<instance part="J2" gate="J$1" x="204.47" y="429.26" smashed="yes">
+<attribute name="VALUE" x="201.93" y="421.894" size="1.778" layer="96" font="vector"/>
+<attribute name="NAME" x="201.93" y="434.848" size="1.778" layer="95" font="vector"/>
 </instance>
 </instances>
@@
 <label x="260.35" y="398.78" size="1.778" layer="95"/>
 </segment>
+<segment>
+<pinref part="J1" gate="G$1" pin="6"/>
+<wire x1="190.5" y1="419.1" x2="182.88" y2="419.1" width="0.1524" layer="91"/>
+<label x="182.88" y="419.1" size="1.778" layer="95"/>
+</segment>
+<segment>
+<pinref part="J2" gate="J$1" pin="1"/>
+<wire x1="212.09" y1="426.72" x2="217.17" y2="426.72" width="0.1524" layer="91"/>
+<label x="217.17" y="426.72" size="1.778" layer="95" rot="R180"/>
+</segment>
 </net>
 <net name="VCC_D" class="0">
@@
 <label x="241.3" y="396.24" size="1.778" layer="95"/>
 </segment>
+<segment>
+<pinref part="J2" gate="J$1" pin="3"/>
+<wire x1="212.09" y1="431.8" x2="217.17" y2="431.8" width="0.1524" layer="91"/>
+<label x="217.17" y="431.8" size="1.778" layer="95" rot="R180"/>
+</segment>
 </net>
 <net name="D10_D" class="0">
@@
 </net>
 <net name="TX_D" class="0">
-<segment>
-<pinref part="JP4" gate="G$1" pin="1"/>
-<wire x1="279.4" y1="367.03" x2="279.4" y2="377.19" width="0.1524" layer="91"/>
-<label x="279.4" y="377.19" size="1.778" layer="95" rot="R270"/>
-</segment>
 <segment>
 <pinref part="U$1" gate="G$1" pin="3"/>
@@
 <label x="247.65" y="402.59" size="1.778" layer="95"/>
 </segment>
-</net>
-<net name="RX_D" class="0">
 <segment>
 <pinref part="JP4" gate="G$1" pin="2"/>
@@
 <label x="276.86" y="377.19" size="1.778" layer="95" rot="R270"/>
 </segment>
+<segment>
+<pinref part="J1" gate="G$1" pin="2"/>
+<wire x1="190.5" y1="429.26" x2="182.88" y2="429.26" width="0.1524" layer="91"/>
+<label x="182.88" y="429.26" size="1.778" layer="95"/>
+</segment>
+</net>
+<net name="RX_D" class="0">
 <segment>
 <pinref part="U$1" gate="G$1" pin="2"/>
@@
 <label x="242.57" y="398.78" size="1.778" layer="95"/>
 </segment>
+<segment>
+<pinref part="JP4" gate="G$1" pin="1"/>
+<wire x1="279.4" y1="367.03" x2="279.4" y2="377.19" width="0.1524" layer="91"/>
+<label x="279.4" y="377.19" size="1.778" layer="95" rot="R270"/>
+</segment>
+<segment>
+<pinref part="J1" gate="G$1" pin="3"/>
+<wire x1="190.5" y1="426.72" x2="182.88" y2="426.72" width="0.1524" layer="91"/>
+<label x="182.88" y="426.72" size="1.778" layer="95"/>
+</segment>
 </net>
 <net name="A6_D" class="0">
@@
 <label x="257.81" y="402.59" size="1.778" layer="95"/>
 </segment>
+<segment>
+<pinref part="J2" gate="J$1" pin="2"/>
+<wire x1="212.09" y1="429.26" x2="217.17" y2="429.26" width="0.1524" layer="91"/>
+<label x="217.17" y="429.26" size="1.778" layer="95" rot="R180"/>
+</segment>
 </net>
 <net name="N$2" class="0">
@@
 </segment>
 </net>
-<net name="N$5" class="0">
-<segment>
-<pinref part="U$2" gate="G$1" pin="1"/>
-<pinref part="J1" gate="G$1" pin="1"/>
-<wire x1="240.03" y1="433.07" x2="245.11" y2="433.07" width="0.1524" layer="91"/>
-</segment>
-</net>
-<net name="N$6" class="0">
-<segment>
-<pinref part="U$2" gate="G$1" pin="2"/>
-<pinref part="J1" gate="G$1" pin="2"/>
-<wire x1="240.03" y1="435.61" x2="245.11" y2="435.61" width="0.1524" layer="91"/>
-</segment>
-</net>
-<net name="N$7" class="0">
-<segment>
-<pinref part="U$2" gate="G$1" pin="3"/>
-<pinref part="J1" gate="G$1" pin="3"/>
-<wire x1="240.03" y1="438.15" x2="245.11" y2="438.15" width="0.1524" layer="91"/>
-</segment>
-</net>
-<net name="N$8" class="0">
-<segment>
-<pinref part="U$2" gate="G$1" pin="4"/>
-<pinref part="J1" gate="G$1" pin="4"/>
-<wire x1="240.03" y1="440.69" x2="245.11" y2="440.69" width="0.1524" layer="91"/>
-</segment>
-</net>
-<net name="N$9" class="0">
-<segment>
-<pinref part="U$2" gate="G$1" pin="5"/>
-<pinref part="J1" gate="G$1" pin="5"/>
-<wire x1="240.03" y1="443.23" x2="245.11" y2="443.23" width="0.1524" layer="91"/>
-</segment>
-</net>
-<net name="N$10" class="0">
-<segment>
-<pinref part="U$2" gate="G$1" pin="6"/>
-<pinref part="J1" gate="G$1" pin="6"/>
-<wire x1="240.03" y1="445.77" x2="245.11" y2="445.77" width="0.1524" layer="91"/>
-</segment>
-</net>
-<net name="N$11" class="0">
-<segment>
-<pinref part="U$2" gate="G$1" pin="7"/>
-<pinref part="J1" gate="G$1" pin="7"/>
-<wire x1="240.03" y1="448.31" x2="245.11" y2="448.31" width="0.1524" layer="91"/>
-</segment>
-</net>
-<net name="N$12" class="0">
-<segment>
-<pinref part="U$2" gate="G$1" pin="8"/>
-<pinref part="J1" gate="G$1" pin="8"/>
-<wire x1="240.03" y1="450.85" x2="245.11" y2="450.85" width="0.1524" layer="91"/>
-</segment>
-</net>
