File: Eagle/JDY-40 Rx/JDY-40 Rx.sch (EAGLE design)
At the start: 13 parts, among them IC1 LD117AV

Commit message: Added Chrome App
Parts:
- removed J3: (no value), SparkFun-Connectors:CONN_03
- removed J6, J8: (no value), SparkFun-Connectors:CONN_02
- removed U$2: 1X8, headers(2mm):1X8
Connections:
- removed net N$10: J1.6, U$2.6
- removed net N$11: J1.7, U$2.7
- removed net N$12: J1.8, U$2.8
- removed net N$5: J1.1, U$2.1
- removed net N$6: J1.2, U$2.2
- removed net N$7: J1.3, U$2.3
- removed net N$8: J1.4, U$2.4
- removed net N$9: J1.5, U$2.5
- net BATT+: no longer J8.1
- net GND_D: no longer J3.2, J6.2
- net RX_D: no longer J6.1
- net TX_D: no longer J3.1
- net VCC_D: no longer J3.3, J8.2
Changed lines of the file:
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@@
 <part name="U$1" library="headers(2mm)" deviceset="1X6" device=""/>
 <part name="D1" library="diode" library_urn="urn:adsk.eagle:library:210" deviceset="1N821" device="" package3d_urn="urn:adsk.eagle:package:43342/1"/>
-<part name="U$2" library="headers(2mm)" deviceset="1X8" device=""/>
 <part name="J1" library="SparkFun-Connectors" library_urn="urn:adsk.eagle:library:513" deviceset="CONN_08" device="&quot;" package3d_urn="urn:adsk.eagle:package:38138/1"/>
 <part name="IC1" library="v-reg" library_urn="urn:adsk.eagle:library:409" deviceset="LD117A?*" device="V" package3d_urn="urn:adsk.eagle:package:30365/1"/>
 <part name="C1" library="SparkFun-Capacitors" deviceset="100UF-POLAR" device="-RADIAL-2.5MM-25V-20%" value="100uF"/>
 <part name="J2" library="SparkFun-Connectors" library_urn="urn:adsk.eagle:library:513" deviceset="CONN_03" device="" package3d_urn="urn:adsk.eagle:package:38063/1"/>
-<part name="J3" library="SparkFun-Connectors" library_urn="urn:adsk.eagle:library:513" deviceset="CONN_03" device="" package3d_urn="urn:adsk.eagle:package:38063/1"/>
 <part name="J4" library="SparkFun-Connectors" library_urn="urn:adsk.eagle:library:513" deviceset="CONN_01" device="" package3d_urn="urn:adsk.eagle:package:38028/1"/>
 <part name="J5" library="SparkFun-Connectors" library_urn="urn:adsk.eagle:library:513" deviceset="CONN_01" device="" package3d_urn="urn:adsk.eagle:package:38028/1"/>
-<part name="J6" library="SparkFun-Connectors" library_urn="urn:adsk.eagle:library:513" deviceset="CONN_02" device="" package3d_urn="urn:adsk.eagle:package:38039/1"/>
 <part name="J7" library="SparkFun-Connectors" library_urn="urn:adsk.eagle:library:513" deviceset="CONN_04" device="" package3d_urn="urn:adsk.eagle:package:38085/1"/>
-<part name="J8" library="SparkFun-Connectors" library_urn="urn:adsk.eagle:library:513" deviceset="CONN_02" device="" package3d_urn="urn:adsk.eagle:package:38039/1"/>
 </parts>
 <sheets>
@@
 <attribute name="NAME" x="212.852" y="426.085" size="1.778" layer="95"/>
 <attribute name="VALUE" x="212.852" y="420.751" size="1.778" layer="96"/>
-</instance>
-<instance part="U$2" gate="G$1" x="247.65" y="443.23" smashed="yes" rot="R180">
-<attribute name="NAME" x="250.19" y="429.895" size="1.27" layer="95" font="vector" rot="R180"/>
-<attribute name="VALUE" x="250.19" y="455.295" size="1.27" layer="96" font="vector" rot="R180"/>
 </instance>
 <instance part="J1" gate="G$1" x="234.95" y="440.69" smashed="yes">
@@
 <attribute name="NAME" x="304.038" y="391.16" size="1.778" layer="95" font="vector" rot="R270"/>
 </instance>
-<instance part="J3" gate="J$1" x="322.58" y="443.23" smashed="yes">
-<attribute name="VALUE" x="320.04" y="435.864" size="1.778" layer="96" font="vector"/>
-<attribute name="NAME" x="320.04" y="448.818" size="1.778" layer="95" font="vector"/>
-</instance>
 <instance part="J4" gate="G$1" x="214.63" y="448.31" smashed="yes" rot="R180">
 <attribute name="VALUE" x="217.17" y="453.136" size="1.778" layer="96" font="vector" rot="R180"/>
@@
 <attribute name="NAME" x="217.17" y="436.372" size="1.778" layer="95" font="vector" rot="R180"/>
 </instance>
-<instance part="J6" gate="G$1" x="322.58" y="403.86" smashed="yes">
-<attribute name="VALUE" x="320.04" y="399.034" size="1.778" layer="96" font="vector"/>
-<attribute name="NAME" x="320.04" y="409.448" size="1.778" layer="95" font="vector"/>
-</instance>
 <instance part="J7" gate="G$1" x="207.01" y="401.32" smashed="yes" rot="R180">
 <attribute name="VALUE" x="212.09" y="408.686" size="1.778" layer="96" font="vector" rot="R180"/>
 <attribute name="NAME" x="212.09" y="393.192" size="1.778" layer="95" font="vector" rot="R180"/>
-</instance>
-<instance part="J8" gate="G$1" x="209.55" y="415.29" smashed="yes" rot="R180">
-<attribute name="VALUE" x="212.09" y="420.116" size="1.778" layer="96" font="vector" rot="R180"/>
-<attribute name="NAME" x="212.09" y="409.702" size="1.778" layer="95" font="vector" rot="R180"/>
 </instance>
 </instances>
@@
 </segment>
 <segment>
-<pinref part="J3" gate="J$1" pin="2"/>
-<wire x1="330.2" y1="443.23" x2="334.01" y2="443.23" width="0.1524" layer="91"/>
-<label x="334.01" y="443.23" size="1.778" layer="95"/>
-</segment>
-<segment>
 <pinref part="J5" gate="G$1" pin="1"/>
 <wire x1="207.01" y1="439.42" x2="199.39" y2="439.42" width="0.1524" layer="91"/>
 <label x="199.39" y="439.42" size="1.778" layer="95"/>
-</segment>
-<segment>
-<pinref part="J6" gate="G$1" pin="2"/>
-<wire x1="330.2" y1="406.4" x2="332.74" y2="406.4" width="0.1524" layer="91"/>
-<label x="332.74" y="406.4" size="1.778" layer="95"/>
 </segment>
 <segment>
@@
 </segment>
 <segment>
-<pinref part="J3" gate="J$1" pin="3"/>
-<wire x1="330.2" y1="445.77" x2="334.01" y2="445.77" width="0.1524" layer="91"/>
-<label x="334.01" y="445.77" size="1.778" layer="95"/>
-</segment>
-<segment>
 <pinref part="J7" gate="G$1" pin="4"/>
 <wire x1="201.93" y1="396.24" x2="195.58" y2="396.24" width="0.1524" layer="91"/>
 <label x="195.58" y="396.24" size="1.778" layer="95"/>
-</segment>
-<segment>
-<pinref part="J8" gate="G$1" pin="2"/>
-<wire x1="201.93" y1="412.75" x2="193.04" y2="412.75" width="0.1524" layer="91"/>
-<label x="193.04" y="412.75" size="1.778" layer="95"/>
 </segment>
 </net>
@@
 <wire x1="255.27" y1="402.59" x2="247.65" y2="402.59" width="0.1524" layer="91"/>
 <label x="247.65" y="402.59" size="1.778" layer="95"/>
-</segment>
-<segment>
-<pinref part="J3" gate="J$1" pin="1"/>
-<wire x1="330.2" y1="440.69" x2="334.01" y2="440.69" width="0.1524" layer="91"/>
-<label x="334.01" y="440.69" size="1.778" layer="95"/>
 </segment>
 <segment>
@@
 </segment>
 <segment>
-<pinref part="J6" gate="G$1" pin="1"/>
-<wire x1="330.2" y1="403.86" x2="332.74" y2="403.86" width="0.1524" layer="91"/>
-<label x="332.74" y="403.86" size="1.778" layer="95"/>
-</segment>
-<segment>
 <pinref part="J7" gate="G$1" pin="1"/>
 <wire x1="201.93" y1="403.86" x2="195.58" y2="403.86" width="0.1524" layer="91"/>
 <label x="195.58" y="403.86" size="1.778" layer="95"/>
-</segment>
-</net>
-<net name="N$5" class="0">
-<segment>
-<pinref part="U$2" gate="G$1" pin="1"/>
-<pinref part="J1" gate="G$1" pin="1"/>
-<wire x1="240.03" y1="433.07" x2="245.11" y2="433.07" width="0.1524" layer="91"/>
-</segment>
-</net>
-<net name="N$6" class="0">
-<segment>
-<pinref part="U$2" gate="G$1" pin="2"/>
-<pinref part="J1" gate="G$1" pin="2"/>
-<wire x1="240.03" y1="435.61" x2="245.11" y2="435.61" width="0.1524" layer="91"/>
-</segment>
-</net>
-<net name="N$7" class="0">
-<segment>
-<pinref part="U$2" gate="G$1" pin="3"/>
-<pinref part="J1" gate="G$1" pin="3"/>
-<wire x1="240.03" y1="438.15" x2="245.11" y2="438.15" width="0.1524" layer="91"/>
-</segment>
-</net>
-<net name="N$8" class="0">
-<segment>
-<pinref part="U$2" gate="G$1" pin="4"/>
-<pinref part="J1" gate="G$1" pin="4"/>
-<wire x1="240.03" y1="440.69" x2="245.11" y2="440.69" width="0.1524" layer="91"/>
-</segment>
-</net>
-<net name="N$9" class="0">
-<segment>
-<pinref part="U$2" gate="G$1" pin="5"/>
-<pinref part="J1" gate="G$1" pin="5"/>
-<wire x1="240.03" y1="443.23" x2="245.11" y2="443.23" width="0.1524" layer="91"/>
-</segment>
-</net>
-<net name="N$10" class="0">
-<segment>
-<pinref part="U$2" gate="G$1" pin="6"/>
-<pinref part="J1" gate="G$1" pin="6"/>
-<wire x1="240.03" y1="445.77" x2="245.11" y2="445.77" width="0.1524" layer="91"/>
-</segment>
-</net>
-<net name="N$11" class="0">
-<segment>
-<pinref part="U$2" gate="G$1" pin="7"/>
-<pinref part="J1" gate="G$1" pin="7"/>
-<wire x1="240.03" y1="448.31" x2="245.11" y2="448.31" width="0.1524" layer="91"/>
-</segment>
-</net>
-<net name="N$12" class="0">
-<segment>
-<pinref part="U$2" gate="G$1" pin="8"/>
-<pinref part="J1" gate="G$1" pin="8"/>
-<wire x1="240.03" y1="450.85" x2="245.11" y2="450.85" width="0.1524" layer="91"/>
 </segment>
 </net>
@@
 <label x="199.39" y="424.18" size="1.778" layer="95"/>
 </segment>
-<segment>
-<pinref part="J8" gate="G$1" pin="1"/>
-<wire x1="201.93" y1="415.29" x2="193.04" y2="415.29" width="0.1524" layer="91"/>
-<label x="193.04" y="415.29" size="1.778" layer="95"/>
-</segment>
 </net>

Commit message: eagle pcb-40 rx
Parts:
- added U$2, U$3, U$4, U$5, U$6, U$7, U$8, U$9: 1X1, headers(2mm):1X1
Connections:
- new net N$1: J1.1, U$2.1
- new net N$2: J1.2, U$3.1
- new net N$3: J1.3, U$4.1
- new net N$4: J1.4, U$5.1
- new net N$5: J1.5, U$6.1
- new net N$6: J1.6, U$7.1
- new net N$7: J1.7, U$8.1
- new net N$8: J1.8, U$9.1
Changed lines of the file:
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@@
 <part name="J5" library="SparkFun-Connectors" library_urn="urn:adsk.eagle:library:513" deviceset="CONN_01" device="" package3d_urn="urn:adsk.eagle:package:38028/1"/>
 <part name="J7" library="SparkFun-Connectors" library_urn="urn:adsk.eagle:library:513" deviceset="CONN_04" device="" package3d_urn="urn:adsk.eagle:package:38085/1"/>
+<part name="U$2" library="headers(2mm)" deviceset="1X1" device=""/>
+<part name="U$3" library="headers(2mm)" deviceset="1X1" device=""/>
+<part name="U$4" library="headers(2mm)" deviceset="1X1" device=""/>
+<part name="U$5" library="headers(2mm)" deviceset="1X1" device=""/>
+<part name="U$6" library="headers(2mm)" deviceset="1X1" device=""/>
+<part name="U$7" library="headers(2mm)" deviceset="1X1" device=""/>
+<part name="U$8" library="headers(2mm)" deviceset="1X1" device=""/>
+<part name="U$9" library="headers(2mm)" deviceset="1X1" device=""/>
 </parts>
 <sheets>
@@
 <attribute name="NAME" x="212.09" y="393.192" size="1.778" layer="95" font="vector" rot="R180"/>
 </instance>
+<instance part="U$2" gate="G$1" x="240.03" y="426.72" smashed="yes" rot="R90">
+<attribute name="NAME" x="236.855" y="424.18" size="1.27" layer="95" font="vector" rot="R90"/>
+<attribute name="VALUE" x="244.475" y="424.18" size="1.27" layer="96" font="vector" rot="R90"/>
+</instance>
+<instance part="U$3" gate="G$1" x="245.11" y="435.61" smashed="yes" rot="R180">
+<attribute name="NAME" x="247.65" y="432.435" size="1.27" layer="95" font="vector" rot="R180"/>
+<attribute name="VALUE" x="247.65" y="440.055" size="1.27" layer="96" font="vector" rot="R180"/>
+</instance>
+<instance part="U$4" gate="G$1" x="254" y="438.15" smashed="yes" rot="R180">
+<attribute name="NAME" x="256.54" y="434.975" size="1.27" layer="95" font="vector" rot="R180"/>
+<attribute name="VALUE" x="256.54" y="442.595" size="1.27" layer="96" font="vector" rot="R180"/>
+</instance>
+<instance part="U$5" gate="G$1" x="245.11" y="440.69" smashed="yes" rot="R180">
+<attribute name="NAME" x="247.65" y="437.515" size="1.27" layer="95" font="vector" rot="R180"/>
+<attribute name="VALUE" x="247.65" y="445.135" size="1.27" layer="96" font="vector" rot="R180"/>
+</instance>
+<instance part="U$6" gate="G$1" x="254" y="443.23" smashed="yes" rot="R180">
+<attribute name="NAME" x="256.54" y="440.055" size="1.27" layer="95" font="vector" rot="R180"/>
+<attribute name="VALUE" x="256.54" y="447.675" size="1.27" layer="96" font="vector" rot="R180"/>
+</instance>
+<instance part="U$7" gate="G$1" x="245.11" y="445.77" smashed="yes" rot="R180">
+<attribute name="NAME" x="247.65" y="442.595" size="1.27" layer="95" font="vector" rot="R180"/>
+<attribute name="VALUE" x="247.65" y="450.215" size="1.27" layer="96" font="vector" rot="R180"/>
+</instance>
+<instance part="U$8" gate="G$1" x="254" y="448.31" smashed="yes" rot="R180">
+<attribute name="NAME" x="256.54" y="445.135" size="1.27" layer="95" font="vector" rot="R180"/>
+<attribute name="VALUE" x="256.54" y="452.755" size="1.27" layer="96" font="vector" rot="R180"/>
+</instance>
+<instance part="U$9" gate="G$1" x="240.03" y="457.2" smashed="yes" rot="R270">
+<attribute name="NAME" x="243.205" y="459.74" size="1.27" layer="95" font="vector" rot="R270"/>
+<attribute name="VALUE" x="235.585" y="459.74" size="1.27" layer="96" font="vector" rot="R270"/>
+</instance>
 </instances>
 <busses>
@@
 </segment>
 </net>
+<net name="N$1" class="0">
+<segment>
+<pinref part="J1" gate="G$1" pin="1"/>
+<pinref part="U$2" gate="G$1" pin="1"/>
+<wire x1="240.03" y1="429.26" x2="240.03" y2="433.07" width="0.1524" layer="91"/>
+</segment>
+</net>
+<net name="N$2" class="0">
+<segment>
+<pinref part="J1" gate="G$1" pin="2"/>
+<pinref part="U$3" gate="G$1" pin="1"/>
+<wire x1="242.57" y1="435.61" x2="240.03" y2="435.61" width="0.1524" layer="91"/>
+</segment>
+</net>
+<net name="N$3" class="0">
+<segment>
+<pinref part="J1" gate="G$1" pin="3"/>
+<pinref part="U$4" gate="G$1" pin="1"/>
+<wire x1="251.46" y1="438.15" x2="240.03" y2="438.15" width="0.1524" layer="91"/>
+</segment>
+</net>
+<net name="N$4" class="0">
+<segment>
+<pinref part="J1" gate="G$1" pin="4"/>
+<pinref part="U$5" gate="G$1" pin="1"/>
+<wire x1="242.57" y1="440.69" x2="240.03" y2="440.69" width="0.1524" layer="91"/>
+</segment>
+</net>
+<net name="N$5" class="0">
+<segment>
+<pinref part="J1" gate="G$1" pin="5"/>
+<pinref part="U$6" gate="G$1" pin="1"/>
+<wire x1="251.46" y1="443.23" x2="240.03" y2="443.23" width="0.1524" layer="91"/>
+</segment>
+</net>
+<net name="N$6" class="0">
+<segment>
+<pinref part="J1" gate="G$1" pin="6"/>
+<pinref part="U$7" gate="G$1" pin="1"/>
+<wire x1="242.57" y1="445.77" x2="240.03" y2="445.77" width="0.1524" layer="91"/>
+</segment>
+</net>
+<net name="N$7" class="0">
+<segment>
+<pinref part="J1" gate="G$1" pin="7"/>
+<pinref part="U$8" gate="G$1" pin="1"/>
+<wire x1="251.46" y1="448.31" x2="240.03" y2="448.31" width="0.1524" layer="91"/>
+</segment>
+</net>
+<net name="N$8" class="0">
+<segment>
+<pinref part="J1" gate="G$1" pin="8"/>
+<pinref part="U$9" gate="G$1" pin="1"/>
+<wire x1="240.03" y1="454.66" x2="240.03" y2="450.85" width="0.1524" layer="91"/>
+</segment>
+</net>
