File: Eagle/wemosRx/wemosRx.brd (EAGLE design)
At the start: 30.1 x 40.6 mm, 3 parts

Commit message: yo
Parts:
- added C1: 100uF, SparkFun-Capacitors:CPOL-RADIAL-2.5MM-6.5MM
- added IC1: LD117AV18, v-reg:TO220L1
Connections:
- net 3.3V: now also C1.1, IC1.2
- net GND: now also C1.2, IC1.1
- net VCC: now also IC1.3; no longer JP3.8
Routing:
- net 3.3V: track 0.00 -> 54.7 mm
- net GND: track 25.4 -> 64.7 mm
- net VCC: track 20.3 -> 41.5 mm
- net D11: track 35.9 -> 47.9 mm
Other:
- board size 30.1 x 40.6 mm -> 30.1 x 44.4 mm
- board text added: "Gnd"
- board text added: "VCC"
- board text removed: "+"
- board text removed: "-"
Changed lines of the file:
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@@
 <?xml version="1.0" encoding="utf-8"?>
 <!DOCTYPE eagle SYSTEM "eagle.dtd">
-<eagle version="9.5.1">
+<eagle version="9.6.1">
 <drawing>
 <settings>
@@
 <layer number="116" name="Patch_BOT" color="9" fill="4" visible="no" active="yes"/>
 <layer number="118" name="Rect_Pads" color="7" fill="1" visible="yes" active="yes"/>
-<layer number="121" name="_tsilk" color="7" fill="1" visible="no" active="yes"/>
+<layer number="121" name="_tsilk" color="7" fill="1" visible="yes" active="yes"/>
 <layer number="122" name="_bsilk" color="7" fill="1" visible="no" active="yes"/>
 <layer number="123" name="tTestmark" color="7" fill="1" visible="no" active="yes"/>
@@
 <board>
 <plain>
-<wire x1="46.66" y1="27.93" x2="46.66" y2="68.57" width="0" layer="20"/>
-<wire x1="46.66" y1="68.57" x2="16.51" y2="68.57" width="0" layer="20"/>
-<wire x1="16.51" y1="68.57" x2="16.51" y2="27.93" width="0" layer="20"/>
+<wire x1="46.66" y1="27.93" x2="46.66" y2="72.38" width="0" layer="20"/>
+<wire x1="46.66" y1="72.38" x2="16.51" y2="72.38" width="0" layer="20"/>
+<wire x1="16.51" y1="72.38" x2="16.51" y2="27.93" width="0" layer="20"/>
 <wire x1="46.66" y1="27.93" x2="16.51" y2="27.93" width="0" layer="20"/>
-<text x="25.4" y="63.5" size="2.1844" layer="1">Antenna</text>
-<text x="40.64" y="29.21" size="2.54" layer="1" rot="R90">+</text>
-<text x="32.258" y="34.29" size="2.54" layer="1">-</text>
-<text x="26.67" y="53.34" size="2.1844" layer="1">Wemos</text>
+<text x="25.4" y="63.5" size="2.1844" layer="121">Antenna</text>
+<text x="45.72" y="31.75" size="2.54" layer="121" rot="R180">VCC</text>
+<text x="32.258" y="34.29" size="2.54" layer="121">Gnd</text>
+<text x="26.67" y="53.34" size="2.1844" layer="121">Wemos</text>
 </plain>
 <attributes>
@@
 <attribute name="VALUE" x="26.67" y="26.67" size="1.27" layer="27"/>
 </element>
+<element name="IC1" library="v-reg" library_urn="urn:adsk.eagle:library:409" package="TO220L1" package3d_urn="urn:adsk.eagle:package:30365/1" value="LD117AV18" x="27.94" y="73.66" smashed="yes">
+<attribute name="NAME" x="24.13" y="78.74" size="1.778" layer="25" ratio="10"/>
+<attribute name="POPULARITY" value="0" x="27.94" y="73.66" size="1.778" layer="27" display="off"/>
+<attribute name="VALUE" x="24.003" y="76.2" size="1.778" layer="27" ratio="10"/>
+</element>
+<element name="C1" library="SparkFun-Capacitors" package="CPOL-RADIAL-2.5MM-6.5MM" value="100uF" x="41.91" y="67.31" smashed="yes">
+<attribute name="NAME" x="41.91" y="70.739" size="0.6096" layer="25" font="vector" ratio="20" align="bottom-center"/>
+<attribute name="PROD_ID" value="CAP-08439" x="41.91" y="67.31" size="1.778" layer="27" display="off"/>
+<attribute name="VALUE" x="41.91" y="63.881" size="0.6096" layer="27" font="vector" ratio="20" align="top-center"/>
+</element>
 </elements>
 <signals>
@@
 <contactref element="JP3" pad="7"/>
 <contactref element="ALTCOMM" pad="3"/>
+<contactref element="IC1" pad="1"/>
+<contactref element="C1" pad="2"/>
+<wire x1="27.94" y1="67.31" x2="25.4" y2="69.85" width="0.1524" layer="16"/>
+<wire x1="40.66" y1="67.31" x2="27.94" y2="67.31" width="0.1524" layer="16"/>
 <wire x1="33.02" y1="45.72" x2="33.02" y2="30.48" width="0.1524" layer="16"/>
 <wire x1="43.18" y1="45.72" x2="33.02" y2="45.72" width="0.1524" layer="16"/>
+<wire x1="40.64" y1="47.625" x2="40.64" y2="67.31" width="0.1524" layer="1"/>
+<wire x1="42.545" y1="45.72" x2="40.64" y2="47.625" width="0.1524" layer="1"/>
+<wire x1="43.18" y1="45.72" x2="42.545" y2="45.72" width="0.1524" layer="1"/>
+<wire x1="40.64" y1="67.31" x2="40.66" y2="67.31" width="0.1524" layer="1"/>
 </signal>
 <signal name="VCC">
-<contactref element="JP3" pad="8"/>
 <contactref element="ALTCOMM" pad="4"/>
-<wire x1="35.56" y1="43.18" x2="35.56" y2="30.48" width="0.1524" layer="16"/>
-<wire x1="43.18" y1="43.18" x2="35.56" y2="43.18" width="0.1524" layer="16"/>
+<contactref element="IC1" pad="3"/>
+<wire x1="35.56" y1="64.77" x2="30.48" y2="69.85" width="0.1524" layer="1"/>
+<wire x1="35.56" y1="30.48" x2="35.56" y2="64.77" width="0.1524" layer="1"/>
 </signal>
 <signal name="3.3V">
 <contactref element="JP5" pad="1"/>
+<contactref element="IC1" pad="2"/>
+<contactref element="C1" pad="1"/>
+<wire x1="29.845" y1="71.755" x2="27.94" y2="69.85" width="0.1524" layer="1"/>
+<wire x1="42.545" y1="71.755" x2="29.845" y2="71.755" width="0.1524" layer="1"/>
+<wire x1="42.545" y1="67.31" x2="42.545" y2="71.755" width="0.1524" layer="1"/>
+<wire x1="42.545" y1="67.31" x2="43.16" y2="67.31" width="0.1524" layer="1"/>
+<wire x1="27.94" y1="43.18" x2="20.32" y2="43.18" width="0.1524" layer="1"/>
+<wire x1="27.94" y1="69.85" x2="27.94" y2="43.18" width="0.1524" layer="1"/>
 </signal>
 <signal name="RST">
@@
 <contactref element="JP3" pad="1"/>
 <contactref element="ALTCOMM" pad="2"/>
-<wire x1="31.115" y1="31.115" x2="30.48" y2="30.48" width="0.1524" layer="1"/>
-<wire x1="31.115" y1="45.4025" x2="31.115" y2="31.115" width="0.1524" layer="1"/>
-<wire x1="40.9575" y1="55.245" x2="31.115" y2="45.4025" width="0.1524" layer="1"/>
-<wire x1="40.9575" y1="59.055" x2="40.9575" y2="55.245" width="0.1524" layer="1"/>
-<wire x1="42.8625" y1="60.96" x2="40.9575" y2="59.055" width="0.1524" layer="1"/>
-<wire x1="43.18" y1="60.96" x2="42.8625" y2="60.96" width="0.1524" layer="1"/>
+<wire x1="30.48" y1="57.15" x2="30.48" y2="30.48" width="0.1524" layer="16"/>
+<wire x1="45.085" y1="57.15" x2="30.48" y2="57.15" width="0.1524" layer="16"/>
+<wire x1="45.72" y1="57.785" x2="45.085" y2="57.15" width="0.1524" layer="16"/>
+<wire x1="45.72" y1="60.96" x2="45.72" y2="57.785" width="0.1524" layer="16"/>
+<wire x1="43.18" y1="60.96" x2="45.72" y2="60.96" width="0.1524" layer="16"/>
 </signal>
 <signal name="D10">
@@
 </board>
 </drawing>
+<compatibility>
+<note version="8.2" severity="warning">
+Since Version 8.2, EAGLE supports online libraries. The ids
+of those online libraries will not be understood (or retained)
+with this version.
+</note>
+<note version="8.3" severity="warning">
+Since Version 8.3, EAGLE supports URNs for individual library
+assets (packages, symbols, and devices). The URNs of those assets
+will not be understood (or retained) with this version.
+</note>
+<note version="8.3" severity="warning">
+Since Version 8.3, EAGLE supports the association of 3D packages
+with devices in libraries, schematics, and board files. Those 3D
+packages will not be understood (or retained) with this version.
+</note>
+</compatibility>
 </eagle>

Commit message: forward
Parts:
- added J1: (no value), SparkFun-Connectors:1X02
- added Q1: 2N5088, transistor-npn:TO92
- added R1: 1K, resistor-power:RS1/4
- added R2: 10K, resistor-power:RS1/4
- moved IC1 14.2 mm to (40.6, 80.0)
- moved ALTCOMM 3.81 mm to (31.8, 30.5)
- turned C1 to 90 degrees
Connections:
- removed net D10: ALTCOMM.1, JP3.2
- new net 5V: J1.2, JP3.8
- new net N$1: Q1.2, R1.2
- new net RX: JP3.2, Q1.3, R2.2
- new net RX_IN: ALTCOMM.1, R1.1
- net 3.3V: now also Q1.1
- net GND: now also R2.1
- net VCC: now also J1.1
Routing:
- net RX_IN: track 0.00 -> 54.4 mm
- net D10: track 43.2 -> 0.00 mm
- net GND: track 64.7 -> 93.1 mm
- net D11: track 47.9 -> 73.6 mm
- net 5V: track 0.00 -> 25.6 mm
- net RX: track 0.00 -> 22.4 mm
- net VCC: track 41.5 -> 63.7 mm
- net 3.3V: track 54.7 -> 64.4 mm
- net N$1: track 0.00 -> 1.90 mm
Other:
- board size 30.1 x 44.4 mm -> 30.1 x 53.3 mm
- board text added: "10K"
- board text added: "1K"
- board text added: "3.3V"
- board text added: "5V"
- board text removed: "Antenna"
