File: Eagle/wemosRx/wemosRx.sch (EAGLE design)
At the start: 3 parts

Commit message: yo
Parts:
- added C1: 100uF, SparkFun-Capacitors:100UF-POLAR-RADIAL-2.5MM-25V-20%
- added IC1: LD117AV18, v-reg:LD117AV18
Connections:
- net 3.3V: now also C1.+, IC1.OUT
- net GND: now also C1.-, IC1.ADJ
- net VCC: now also IC1.IN; no longer JP3.8
Changed lines of the file:
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@@
 <?xml version="1.0" encoding="utf-8"?>
 <!DOCTYPE eagle SYSTEM "eagle.dtd">
-<eagle version="9.5.1">
+<eagle version="9.6.1">
 <drawing>
 <settings>
@@
 <part name="JP5" library="SparkFun-Connectors" deviceset="M08" device="LONGPADS"/>
 <part name="JP3" library="SparkFun-Connectors" deviceset="M08" device="LONGPADS"/>
-<part name="P+2" library="SparkFun" deviceset="VCC" device=""/>
 <part name="GND2" library="SparkFun" deviceset="GND" device=""/>
 <part name="ALTCOMM" library="SparkFun-Connectors" deviceset="M04" device="LONGPADS"/>
 <part name="P+3" library="SparkFun" deviceset="VCC" device=""/>
 <part name="GND4" library="SparkFun" deviceset="GND" device=""/>
+<part name="IC1" library="v-reg" library_urn="urn:adsk.eagle:library:409" deviceset="LD117A?*" device="V" package3d_urn="urn:adsk.eagle:package:30365/1" technology="18"/>
+<part name="GND1" library="SparkFun" deviceset="GND" device=""/>
+<part name="C1" library="SparkFun-Capacitors" deviceset="100UF-POLAR" device="-RADIAL-2.5MM-25V-20%" value="100uF"/>
+<part name="GND3" library="SparkFun" deviceset="GND" device=""/>
+<part name="P+1" library="SparkFun" deviceset="VCC" device=""/>
 </parts>
 <sheets>
@@
 <attribute name="NAME" x="6.35" y="178.308" size="1.778" layer="95" rot="R180"/>
 </instance>
-<instance part="P+2" gate="1" x="-7.62" y="181.61" smashed="yes" rot="R90">
-<attribute name="VALUE" x="-11.176" y="180.594" size="1.778" layer="96" rot="R90"/>
-</instance>
 <instance part="GND2" gate="1" x="-17.78" y="184.15" smashed="yes" rot="R270">
 <attribute name="VALUE" x="-20.32" y="186.69" size="1.778" layer="96" rot="R270"/>
@@
 <instance part="GND4" gate="1" x="27.94" y="172.72" smashed="yes">
 <attribute name="VALUE" x="25.4" y="170.18" size="1.778" layer="96"/>
+</instance>
+<instance part="IC1" gate="G$1" x="-27.94" y="233.68" smashed="yes">
+<attribute name="NAME" x="-25.4" y="226.06" size="1.778" layer="95"/>
+<attribute name="VALUE" x="-25.4" y="223.52" size="1.778" layer="96"/>
+</instance>
+<instance part="GND1" gate="1" x="-27.94" y="220.98" smashed="yes">
+<attribute name="VALUE" x="-30.48" y="218.44" size="1.778" layer="96"/>
+</instance>
+<instance part="C1" gate="G$1" x="12.7" y="232.41" smashed="yes">
+<attribute name="NAME" x="13.716" y="233.045" size="1.778" layer="95" font="vector"/>
+<attribute name="VALUE" x="13.716" y="228.219" size="1.778" layer="96" font="vector"/>
+</instance>
+<instance part="GND3" gate="1" x="6.35" y="227.33" smashed="yes" rot="R270">
+<attribute name="VALUE" x="3.81" y="229.87" size="1.778" layer="96" rot="R270"/>
+</instance>
+<instance part="P+1" gate="1" x="-39.37" y="233.68" smashed="yes" rot="R90">
+<attribute name="VALUE" x="-42.926" y="232.664" size="1.778" layer="96" rot="R90"/>
 </instance>
 </instances>
@@
 <wire x1="27.94" y1="175.26" x2="27.94" y2="181.61" width="0.1524" layer="91"/>
 </segment>
+<segment>
+<pinref part="IC1" gate="G$1" pin="ADJ"/>
+<pinref part="GND1" gate="1" pin="GND"/>
+<wire x1="-27.94" y1="223.52" x2="-27.94" y2="226.06" width="0.1524" layer="91"/>
+</segment>
+<segment>
+<pinref part="C1" gate="G$1" pin="-"/>
+<pinref part="GND3" gate="1" pin="GND"/>
+<wire x1="8.89" y1="227.33" x2="12.7" y2="227.33" width="0.1524" layer="91"/>
+</segment>
 </net>
 <net name="VCC" class="0">
-<segment>
-<pinref part="JP3" gate="G$1" pin="8"/>
-<pinref part="P+2" gate="1" pin="VCC"/>
-<wire x1="-7.62" y1="181.61" x2="-3.81" y2="181.61" width="0.1524" layer="91"/>
-</segment>
 <segment>
 <pinref part="ALTCOMM" gate="G$1" pin="4"/>
@@
 <wire x1="30.48" y1="168.91" x2="30.48" y2="181.61" width="0.1524" layer="91"/>
 </segment>
+<segment>
+<pinref part="IC1" gate="G$1" pin="IN"/>
+<pinref part="P+1" gate="1" pin="VCC"/>
+<wire x1="-39.37" y1="233.68" x2="-35.56" y2="233.68" width="0.1524" layer="91"/>
+</segment>
 </net>
 <net name="3.3V" class="0">
@@
 <wire x1="-46.99" y1="181.61" x2="-43.18" y2="181.61" width="0.1524" layer="91"/>
 <label x="-43.18" y="181.61" size="1.778" layer="95"/>
+</segment>
+<segment>
+<pinref part="IC1" gate="G$1" pin="OUT"/>
+<wire x1="-20.32" y1="233.68" x2="-16.51" y2="233.68" width="0.1524" layer="91"/>
+<label x="-16.51" y="233.68" size="1.778" layer="95"/>
+</segment>
+<segment>
+<pinref part="C1" gate="G$1" pin="+"/>
+<wire x1="12.7" y1="234.95" x2="3.81" y2="234.95" width="0.1524" layer="91"/>
+<label x="3.81" y="234.95" size="1.778" layer="95"/>
 </segment>
 </net>
@@
 </schematic>
 </drawing>
+<compatibility>
+<note version="8.2" severity="warning">
+Since Version 8.2, EAGLE supports online libraries. The ids
+of those online libraries will not be understood (or retained)
+with this version.
+</note>
+<note version="8.3" severity="warning">
+Since Version 8.3, EAGLE supports URNs for individual library
+assets (packages, symbols, and devices). The URNs of those assets
+will not be understood (or retained) with this version.
+</note>
+<note version="8.3" severity="warning">
+Since Version 8.3, EAGLE supports the association of 3D packages
+with devices in libraries, schematics, and board files. Those 3D
+packages will not be understood (or retained) with this version.
+</note>
+</compatibility>
 </eagle>

Commit message: forward
Parts:
- added J1: (no value), SparkFun-Connectors:CONN_02
- added Q1: 2N5088, transistor-npn:2N5088
- added R1: 1K, resistor-power:RRS1/4
- added R2: 10K, resistor-power:RRS1/4
Connections:
- removed net D10: ALTCOMM.1, JP3.2
- new net 5V: J1.2, JP3.8
- new net N$1: Q1.B, R1.2
- new net RX: JP3.2, Q1.E, R2.2
- new net RX_IN: ALTCOMM.1, R1.1
- net 3.3V: now also Q1.C
- net GND: now also R2.1
- net VCC: now also J1.1
Changed lines of the file:
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@@
 <part name="GND3" library="SparkFun" deviceset="GND" device=""/>
 <part name="P+1" library="SparkFun" deviceset="VCC" device=""/>
+<part name="GND5" library="SparkFun" deviceset="GND" device=""/>
+<part name="Q1" library="transistor-npn" library_urn="urn:adsk.eagle:library:398" deviceset="2N5088" device="" package3d_urn="urn:adsk.eagle:package:28523/2"/>
+<part name="R1" library="resistor-power" library_urn="urn:adsk.eagle:library:344" deviceset="R" device="RS1/4" package3d_urn="urn:adsk.eagle:package:25167/1" value="1K"/>
+<part name="R2" library="resistor-power" library_urn="urn:adsk.eagle:library:344" deviceset="R" device="RS1/4" package3d_urn="urn:adsk.eagle:package:25167/1" value="10K"/>
+<part name="J1" library="SparkFun-Connectors" deviceset="CONN_02" device=""/>
 </parts>
 <sheets>
@@
 <attribute name="VALUE" x="-42.926" y="232.664" size="1.778" layer="96" rot="R90"/>
 </instance>
+<instance part="GND5" gate="1" x="43.18" y="201.93" smashed="yes">
+<attribute name="VALUE" x="40.64" y="199.39" size="1.778" layer="96"/>
+</instance>
+<instance part="Q1" gate="G$1" x="40.64" y="223.52" smashed="yes">
+<attribute name="NAME" x="30.48" y="231.14" size="1.778" layer="95"/>
+<attribute name="VALUE" x="30.48" y="228.6" size="1.778" layer="96"/>
+</instance>
+<instance part="R1" gate="G$1" x="30.48" y="223.52" smashed="yes">
+<attribute name="NAME" x="26.67" y="224.8916" size="1.778" layer="95"/>
+<attribute name="VALUE" x="26.67" y="220.599" size="1.778" layer="96"/>
+</instance>
+<instance part="R2" gate="G$1" x="43.18" y="212.09" smashed="yes" rot="R90">
+<attribute name="NAME" x="41.8084" y="208.28" size="1.778" layer="95" rot="R90"/>
+<attribute name="VALUE" x="46.101" y="208.28" size="1.778" layer="96" rot="R90"/>
+</instance>
+<instance part="J1" gate="G$1" x="-3.81" y="243.84" smashed="yes">
+<attribute name="VALUE" x="-6.35" y="239.014" size="1.778" layer="96" font="vector"/>
+<attribute name="NAME" x="-6.35" y="249.428" size="1.778" layer="95" font="vector"/>
+</instance>
 </instances>
 <busses>
@@
 <wire x1="8.89" y1="227.33" x2="12.7" y2="227.33" width="0.1524" layer="91"/>
 </segment>
+<segment>
+<pinref part="R2" gate="G$1" pin="1"/>
+<pinref part="GND5" gate="1" pin="GND"/>
+<wire x1="43.18" y1="204.47" x2="43.18" y2="207.01" width="0.1524" layer="91"/>
+</segment>
 </net>
 <net name="VCC" class="0">
@@
 <wire x1="-39.37" y1="233.68" x2="-35.56" y2="233.68" width="0.1524" layer="91"/>
 </segment>
+<segment>
+<pinref part="J1" gate="G$1" pin="1"/>
+<wire x1="3.81" y1="243.84" x2="10.16" y2="243.84" width="0.1524" layer="91"/>
+<label x="10.16" y="243.84" size="1.778" layer="95" rot="R180"/>
+</segment>
 </net>
 <net name="3.3V" class="0">
@@
 <label x="3.81" y="234.95" size="1.778" layer="95"/>
 </segment>
+<segment>
+<pinref part="Q1" gate="G$1" pin="C"/>
+<wire x1="43.18" y1="228.6" x2="43.18" y2="237.49" width="0.1524" layer="91"/>
+<label x="43.18" y="237.49" size="1.778" layer="95"/>
+</segment>
 </net>
 <net name="RST" class="0">
@@
 </segment>
 </net>
-<net name="D10" class="0">
+<net name="D1" class="0">
+<segment>
+<pinref part="JP3" gate="G$1" pin="3"/>
+<wire x1="-3.81" y1="194.31" x2="-11.43" y2="194.31" width="0.1524" layer="91"/>
+<label x="-11.43" y="194.31" size="1.778" layer="95"/>
+</segment>
+</net>
+<net name="D2" class="0">
+<segment>
+<pinref part="JP3" gate="G$1" pin="4"/>
+<wire x1="-3.81" y1="191.77" x2="-11.43" y2="191.77" width="0.1524" layer="91"/>
+<label x="-11.43" y="191.77" size="1.778" layer="95"/>
+</segment>
+</net>
+<net name="D3" class="0">
+<segment>
+<pinref part="JP3" gate="G$1" pin="5"/>
+<wire x1="-3.81" y1="189.23" x2="-11.43" y2="189.23" width="0.1524" layer="91"/>
+<label x="-11.43" y="189.23" size="1.778" layer="95"/>
+</segment>
+</net>
+<net name="D4" class="0">
+<segment>
+<pinref part="JP3" gate="G$1" pin="6"/>
+<wire x1="-3.81" y1="186.69" x2="-11.43" y2="186.69" width="0.1524" layer="91"/>
+<label x="-11.43" y="186.69" size="1.778" layer="95"/>
+</segment>
+</net>
+<net name="A0" class="0">
+<segment>
+<pinref part="JP5" gate="G$1" pin="7"/>
+<wire x1="-46.99" y1="196.85" x2="-43.18" y2="196.85" width="0.1524" layer="91"/>
+<label x="-43.18" y="196.85" size="1.778" layer="95"/>
+</segment>
+</net>
+<net name="D0" class="0">
+<segment>
+<pinref part="JP5" gate="G$1" pin="6"/>
+<wire x1="-46.99" y1="194.31" x2="-43.18" y2="194.31" width="0.1524" layer="91"/>
+<label x="-43.18" y="194.31" size="1.778" layer="95"/>
+</segment>
+</net>
+<net name="D5" class="0">
+<segment>
+<pinref part="JP5" gate="G$1" pin="5"/>
+<wire x1="-46.99" y1="191.77" x2="-43.18" y2="191.77" width="0.1524" layer="91"/>
+<label x="-43.18" y="191.77" size="1.778" layer="95"/>
+</segment>
+</net>
+<net name="D6" class="0">
+<segment>
+<pinref part="JP5" gate="G$1" pin="4"/>
+<wire x1="-46.99" y1="189.23" x2="-43.18" y2="189.23" width="0.1524" layer="91"/>
+<label x="-43.18" y="189.23" size="1.778" layer="95"/>
+</segment>
+</net>
+<net name="D7" class="0">
+<segment>
+<pinref part="JP5" gate="G$1" pin="3"/>
+<wire x1="-46.99" y1="186.69" x2="-43.18" y2="186.69" width="0.1524" layer="91"/>
+<label x="-43.18" y="186.69" size="1.778" layer="95"/>
+</segment>
+</net>
+<net name="N$1" class="0">
+<segment>
+<pinref part="Q1" gate="G$1" pin="B"/>
+<pinref part="R1" gate="G$1" pin="2"/>
+<wire x1="35.56" y1="223.52" x2="38.1" y2="223.52" width="0.1524" layer="91"/>
+</segment>
+</net>
+<net name="RX" class="0">
 <segment>
 <pinref part="JP3" gate="G$1" pin="2"/>
-<wire x1="-3.81" y1="196.85" x2="-19.05" y2="196.85" width="0.1524" layer="91"/>
-<label x="-19.05" y="196.85" size="1.778" layer="95"/>
-</segment>
+<wire x1="-3.81" y1="196.85" x2="-17.78" y2="196.85" width="0.1524" layer="91"/>
+<label x="-17.78" y="196.85" size="1.778" layer="95"/>
+</segment>
+<segment>
+<pinref part="Q1" gate="G$1" pin="E"/>
+<pinref part="R2" gate="G$1" pin="2"/>
+<wire x1="43.18" y1="217.17" x2="43.18" y2="218.44" width="0.1524" layer="91"/>
+<wire x1="43.18" y1="218.44" x2="48.26" y2="218.44" width="0.1524" layer="91"/>
+<junction x="43.18" y="218.44"/>
+<label x="48.26" y="218.44" size="1.778" layer="95"/>
+</segment>
+</net>
+<net name="RX_IN" class="0">
 <segment>
 <pinref part="ALTCOMM" gate="G$1" pin="1"/>
@@
 <label x="15.24" y="181.61" size="1.778" layer="95"/>
 </segment>
-</net>
-<net name="D1" class="0">
-<segment>
-<pinref part="JP3" gate="G$1" pin="3"/>
-<wire x1="-3.81" y1="194.31" x2="-11.43" y2="194.31" width="0.1524" layer="91"/>
-<label x="-11.43" y="194.31" size="1.778" layer="95"/>
-</segment>
-</net>
-<net name="D2" class="0">
-<segment>
-<pinref part="JP3" gate="G$1" pin="4"/>
-<wire x1="-3.81" y1="191.77" x2="-11.43" y2="191.77" width="0.1524" layer="91"/>
-<label x="-11.43" y="191.77" size="1.778" layer="95"/>
-</segment>
-</net>
-<net name="D3" class="0">
-<segment>
-<pinref part="JP3" gate="G$1" pin="5"/>
-<wire x1="-3.81" y1="189.23" x2="-11.43" y2="189.23" width="0.1524" layer="91"/>
-<label x="-11.43" y="189.23" size="1.778" layer="95"/>
-</segment>
-</net>
-<net name="D4" class="0">
-<segment>
-<pinref part="JP3" gate="G$1" pin="6"/>
-<wire x1="-3.81" y1="186.69" x2="-11.43" y2="186.69" width="0.1524" layer="91"/>
-<label x="-11.43" y="186.69" size="1.778" layer="95"/>
-</segment>
-</net>
-<net name="A0" class="0">
-<segment>
-<pinref part="JP5" gate="G$1" pin="7"/>
-<wire x1="-46.99" y1="196.85" x2="-43.18" y2="196.85" width="0.1524" layer="91"/>
-<label x="-43.18" y="196.85" size="1.778" layer="95"/>
-</segment>
-</net>
-<net name="D0" class="0">
-<segment>
-<pinref part="JP5" gate="G$1" pin="6"/>
-<wire x1="-46.99" y1="194.31" x2="-43.18" y2="194.31" width="0.1524" layer="91"/>
-<label x="-43.18" y="194.31" size="1.778" layer="95"/>
-</segment>
-</net>
-<net name="D5" class="0">
-<segment>
-<pinref part="JP5" gate="G$1" pin="5"/>
-<wire x1="-46.99" y1="191.77" x2="-43.18" y2="191.77" width="0.1524" layer="91"/>
-<label x="-43.18" y="191.77" size="1.778" layer="95"/>
-</segment>
-</net>
-<net name="D6" class="0">
-<segment>
-<pinref part="JP5" gate="G$1" pin="4"/>
-<wire x1="-46.99" y1="189.23" x2="-43.18" y2="189.23" width="0.1524" layer="91"/>
-<label x="-43.18" y="189.23" size="1.778" layer="95"/>
-</segment>
-</net>
-<net name="D7" class="0">
-<segment>
-<pinref part="JP5" gate="G$1" pin="3"/>
-<wire x1="-46.99" y1="186.69" x2="-43.18" y2="186.69" width="0.1524" layer="91"/>
-<label x="-43.18" y="186.69" size="1.778" layer="95"/>
-</segment>
-</net>
+<segment>
+<pinref part="R1" gate="G$1" pin="1"/>
+<wire x1="25.4" y1="223.52" x2="16.51" y2="223.52" width="0.1524" layer="91"/>
+<label x="16.51" y="223.52" size="1.778" layer="95"/>
+</segment>
+</net>
+<net name="5V" class="0">
+<segment>
+<pinref part="JP3" gate="G$1" pin="8"/>
+<wire x1="-3.81" y1="181.61" x2="-11.43" y2="181.61" width="0.1524" layer="91"/>
+<label x="-11.43" y="181.61" size="1.778" layer="95"/>
+</segment>
+<segment>
+<pinref part="J1" gate="G$1" pin="2"/>
+<wire x1="3.81" y1="246.38" x2="3.81" y2="255.27" width="0.1524" layer="91"/>
+<label x="3.81" y="255.27" size="1.778" layer="95"/>
+</segment>
+</net>
