File: Eagle/escControl/escControl.sch (EAGLE design)
At the start: 8 parts

Commit message: ddns.net
Parts:
- removed J1, J2: (no value), SparkFun-Connectors:CONN_09
- added J7, J8: (no value), SparkFun-Connectors:CONN_06SILK_FEMALE_PTH
- added U$1, U$2: 1X3, headers(2mm):1X3
Connections:
- removed net N$5: D1.A, J1.8
- removed net N$6: J1.5, J1.6
- new net N$1: D5.A, U$1.2
- new net N$3: D1.A, U$2.2
- net 7.4V: now also J7.4, J8.4; no longer J1.3, J2.3
- net D5: now also U$1.1; no longer J2.9
- net D6: now also U$2.1; no longer J1.9
- net GND: now also J7.1, J8.1, U$1.3, U$2.3; no longer J1.2, J1.7, J2.2, J2.7
- net N$2: now also J7.5, J7.6; no longer D5.A, J2.8
- net N$4: now also J8.5, J8.6; no longer J2.5, J2.6
Other:
- moved on the sheet: D1, D5
