File: Eagle/nanoController/nanoController.sch (EAGLE design)
At the start: 11 parts

Commit message: yo
Parts:
- removed 3.3VOLT: Regulator, SparkFun-Connectors:M03LONGPADS
- removed 5VIN: Power, SparkFun-Connectors:M023.5MM
- removed C1: (no value), SparkFun-Capacitors:10UF-25V-20%(PTH)
- added J1: (no value), SparkFun-Connectors:CONN_06SILK_FEMALE_PTH
- renumbered RECEIVER to WIFI_RECEIVER
Connections:
- removed net 3.3V: 3.3CAM.1, 3.3VOLT.2, C1.+
- net D11: now also J1.5
- net D12: now also J1.6
- net D7: now also J1.2
- net D8: now also J1.1
- net GND: now also J1.4; no longer 3.3VOLT.1, 5VIN.2, C1.-
- net VCC: now also 3.3CAM.1, J1.3; no longer 3.3VOLT.3, 5VIN.1

Commit message: webserver
Parts:
- removed 3.3CAM: Power, SparkFun-Connectors:M023.5MM
- added 3.3CAM1, 3.3CAM2, 3.3CAM3: Power, SparkFun-Connectors:M023.5MM
- added EXTRA: (no value), SparkFun-Connectors:CONN_04LONGPADS
- added GND10, GND11, GND12, GND14: (no value), SparkFun-Connectors:M01PTH_LONGPAD
Connections:
- new net 7.4V: 3.3CAM1.1, 3.3CAM2.1, 3.3CAM3.1, GND10.1
- net D18: now also EXTRA.3
- net D19: now also EXTRA.4
- net GND: now also 3.3CAM1.2, 3.3CAM2.2, 3.3CAM3.2, EXTRA.2, GND12.1, GND14.1; no longer 3.3CAM.2
- net VCC: now also EXTRA.1, GND11.1; no longer 3.3CAM.1
