File: docs/Eagle/piHatMotorDriver/piHatMotorDriver.brd (EAGLE design)
At the start: 78.7 x 56.1 mm, 19 parts, among them Q1 2N5088

Commit message: yo
Parts:
- added J11: (no value), SparkFun-Connectors:1X06
- moved J1 13.2 mm to (25.4, 15.2)
- moved J2 13.2 mm to (25.4, 10.2)
Connections:
- net 7V_B: now also J11.4
- net GND_B: now also J11.3
- net GPIO20: now also J11.2
- net GPIO21: now also J11.1
Routing:
- net GPIO12: track 33.2 -> 152.8 mm
- net GPIO16: track 30.6 -> 149.2 mm
- net GPIO20: track 0.00 -> 93.4 mm
- net GPIO21: track 0.00 -> 90.8 mm
- net GND_B: track 163.2 -> 189.7 mm
- net LREVERSE: track 58.4 -> 38.7 mm
- net LFORWARD: track 51.4 -> 34.2 mm, vias 0 -> 1
- net 7V_B: track 48.6 -> 64.6 mm
- net RFORWARD: track 42.3 -> 50.3 mm
- net RREVERSE: track 50.4 -> 42.5 mm
- net 3.3V_B: track 54.1 -> 49.9 mm, vias 1 -> 0
Other:
- board text added: "+ - Turret"
- board text added: "7V In"
- board text removed: "INPUT"
