File: docs/Eagle/piHatMotorDriver/piHatMotorDriver.sch (EAGLE design)
At the start: 19 parts, among them Q1 2N5088

Commit message: yo
Parts:
- added J11: (no value), SparkFun-Connectors:CONN_06SILK_FEMALE_PTH
Connections:
- net 7V_B: now also J11.4
- net GND_B: now also J11.3
- net GPIO20: now also J11.2
- net GPIO21: now also J11.1
Other:
- note removed: "Fire Relay"
- note removed: "IR Receive"
- note removed: "IR Transmit"
- note removed: "Pixel Data"
- note removed: "Turret Down"
- note removed: "Turret Up"
Changed lines of the file:
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@@
 </classes>
 <parts>
-<part name="GND8" library="SparkFun" deviceset="GND" device=""/>
-<part name="P+5" library="SparkFun" deviceset="VCC" device=""/>
 <part name="J9" library="SparkFun-Connectors" deviceset="CONN_20" device=""/>
 <part name="J10" library="SparkFun-Connectors" deviceset="CONN_20" device=""/>
@@
 <part name="J7" library="SparkFun-Connectors" deviceset="CONN_01" device=""/>
 <part name="J8" library="SparkFun-Connectors" deviceset="CONN_01" device=""/>
+<part name="J11" library="SparkFun-Connectors" deviceset="CONN_06" device="SILK_FEMALE_PTH"/>
 </parts>
 <sheets>
 <sheet>
 <plain>
-<text x="95.25" y="161.29" size="1.778" layer="91">Turret Up</text>
-<text x="95.25" y="158.75" size="1.778" layer="91">Turret Down</text>
-<text x="95.25" y="156.21" size="1.778" layer="91">Fire Relay</text>
-<text x="95.25" y="153.67" size="1.778" layer="91">Pixel Data</text>
-<text x="95.25" y="151.13" size="1.778" layer="91">IR Receive</text>
-<text x="95.25" y="148.59" size="1.778" layer="91">IR Transmit</text>
 <text x="72.39" y="297.18" size="1.778" layer="91" rot="R90">Hit Detected</text>
 <text x="74.93" y="302.26" size="1.778" layer="91" rot="R90">Fire</text>
 </plain>
 <instances>
-<instance part="GND8" gate="1" x="86.36" y="138.43" smashed="yes">
-<attribute name="VALUE" x="83.82" y="135.89" size="1.778" layer="96"/>
-</instance>
-<instance part="P+5" gate="1" x="86.36" y="143.51" smashed="yes" rot="R270">
-<attribute name="VALUE" x="89.916" y="144.526" size="1.778" layer="96" rot="R270"/>
-</instance>
 <instance part="J9" gate="G$1" x="95.25" y="323.85" smashed="yes" rot="R90">
 <attribute name="VALUE" x="94.996" y="323.85" size="1.778" layer="96" font="vector" rot="R90"/>
@@
 <attribute name="VALUE" x="48.26" y="398.526" size="1.778" layer="96" font="vector" rot="R180"/>
 <attribute name="NAME" x="48.26" y="390.652" size="1.778" layer="95" font="vector" rot="R180"/>
+</instance>
+<instance part="J11" gate="G$1" x="118.11" y="271.78" smashed="yes" rot="R90">
+<attribute name="VALUE" x="128.016" y="266.7" size="1.778" layer="96" font="vector" rot="R90"/>
+<attribute name="NAME" x="107.442" y="266.7" size="1.778" layer="95" font="vector" rot="R90"/>
 </instance>
 </instances>
@@
 </busses>
 <nets>
-<net name="GND" class="2">
-<segment>
-<pinref part="GND8" gate="1" pin="GND"/>
-<wire x1="86.36" y1="140.97" x2="77.47" y2="140.97" width="0.1524" layer="91"/>
-</segment>
-</net>
-<net name="D3" class="0">
-<segment>
-<wire x1="77.47" y1="148.59" x2="86.36" y2="148.59" width="0.1524" layer="91"/>
-<label x="86.36" y="148.59" size="1.778" layer="95"/>
-</segment>
-</net>
-<net name="D5" class="0">
-<segment>
-<wire x1="77.47" y1="130.81" x2="82.55" y2="130.81" width="0.1524" layer="91"/>
-<label x="82.55" y="130.81" size="1.778" layer="95"/>
-</segment>
-</net>
-<net name="D6" class="0">
-<segment>
-<wire x1="77.47" y1="128.27" x2="82.55" y2="128.27" width="0.1524" layer="91"/>
-<label x="82.55" y="128.27" size="1.778" layer="95"/>
-</segment>
-</net>
-<net name="D7" class="0">
-<segment>
-<wire x1="77.47" y1="161.29" x2="86.36" y2="161.29" width="0.1524" layer="91"/>
-<label x="86.36" y="161.29" size="1.778" layer="95"/>
-</segment>
-</net>
-<net name="D8" class="0">
-<segment>
-<wire x1="77.47" y1="158.75" x2="86.36" y2="158.75" width="0.1524" layer="91"/>
-<label x="86.36" y="158.75" size="1.778" layer="95"/>
-</segment>
-</net>
-<net name="D9" class="0">
-<segment>
-<wire x1="77.47" y1="125.73" x2="82.55" y2="125.73" width="0.1524" layer="91"/>
-<label x="82.55" y="125.73" size="1.778" layer="95"/>
-</segment>
-</net>
-<net name="D11" class="0">
-<segment>
-<wire x1="77.47" y1="163.83" x2="86.36" y2="163.83" width="0.1524" layer="91"/>
-<label x="86.36" y="163.83" size="1.778" layer="95"/>
-</segment>
-</net>
-<net name="D10" class="0">
-<segment>
-<wire x1="77.47" y1="123.19" x2="82.55" y2="123.19" width="0.1524" layer="91"/>
-<label x="82.55" y="123.19" size="1.778" layer="95"/>
-</segment>
-</net>
-<net name="VCC" class="0">
-<segment>
-<pinref part="P+5" gate="1" pin="VCC"/>
-<wire x1="86.36" y1="143.51" x2="77.47" y2="143.51" width="0.1524" layer="91"/>
-</segment>
-</net>
-<net name="D4" class="0">
-<segment>
-<wire x1="77.47" y1="156.21" x2="86.36" y2="156.21" width="0.1524" layer="91"/>
-<label x="86.36" y="156.21" size="1.778" layer="95"/>
-</segment>
-</net>
-<net name="D2" class="0">
-<segment>
-<wire x1="77.47" y1="153.67" x2="86.36" y2="153.67" width="0.1524" layer="91"/>
-<label x="86.36" y="153.67" size="1.778" layer="95"/>
-</segment>
-</net>
-<net name="D12" class="0">
-<segment>
-<wire x1="77.47" y1="166.37" x2="86.36" y2="166.37" width="0.1524" layer="91"/>
-<label x="86.36" y="166.37" size="1.778" layer="95"/>
-</segment>
-</net>
-<net name="D17" class="0">
-<segment>
-<wire x1="77.47" y1="151.13" x2="86.36" y2="151.13" width="0.1524" layer="91"/>
-<label x="86.36" y="151.13" size="1.778" layer="95"/>
-</segment>
-</net>
-<net name="7.4V" class="0">
-<segment>
-<wire x1="77.47" y1="146.05" x2="86.36" y2="146.05" width="0.1524" layer="91"/>
-<label x="86.36" y="146.05" size="1.778" layer="95"/>
-</segment>
-</net>
 <net name="VCC_B" class="0">
 <segment>
@@
 <label x="-11.43" y="375.92" size="1.778" layer="95"/>
 </segment>
+<segment>
+<pinref part="J11" gate="G$1" pin="3"/>
+<wire x1="118.11" y1="276.86" x2="118.11" y2="285.75" width="0.1524" layer="91"/>
+<label x="118.11" y="285.75" size="1.778" layer="95"/>
+</segment>
 </net>
 <net name="D3_B" class="0">
@@
 <label x="-11.43" y="387.35" size="1.778" layer="95"/>
 </segment>
+<segment>
+<pinref part="J11" gate="G$1" pin="4"/>
+<wire x1="115.57" y1="276.86" x2="115.57" y2="289.56" width="0.1524" layer="91"/>
+<label x="115.57" y="289.56" size="1.778" layer="95"/>
+</segment>
 </net>
 <net name="GPIO20" class="0">
@@
 <label x="87.63" y="336.55" size="1.778" layer="95" rot="R90"/>
 </segment>
+<segment>
+<pinref part="J11" gate="G$1" pin="2"/>
+<wire x1="120.65" y1="276.86" x2="120.65" y2="283.21" width="0.1524" layer="91"/>
+<label x="120.65" y="283.21" size="1.778" layer="95"/>
+</segment>
 </net>
 <net name="GPIO21" class="0">
@@
 <label x="90.17" y="336.55" size="1.778" layer="95" rot="R90"/>
 </segment>
-</net>
+<segment>
+<pinref part="J11" gate="G$1" pin="1"/>
+<wire x1="123.19" y1="276.86" x2="123.19" y2="280.67" width="0.1524" layer="91"/>
+<label x="123.19" y="280.67" size="1.778" layer="95"/>
+</segment>
+</net>
